File: type1/tht/encoder-switch-type1-tht.sch (EAGLE design)
At the start: 9 parts

Commit message: STEP files added, modified modules updated
Parts:
- C1, C2: device 001-private-inventory:CAPACITOR_1025-024X044 -> 006-rcl:CAPACITOR_1025-024X044
- R1, R2, R3, R4, R5: device 001-private-inventory:RESISTOR0204/2V -> 006-rcl:RESISTOR0204/2V
Changed lines of the file:
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@@
 </classes>
 <parts>
-<part name="R1" library="001-private-inventory" deviceset="RESISTOR" device="0204/2V" package3d_urn="urn:adsk.eagle:package:23495/1" value="10K"/>
-<part name="R2" library="001-private-inventory" deviceset="RESISTOR" device="0204/2V" package3d_urn="urn:adsk.eagle:package:23495/1" value="4K7"/>
-<part name="R3" library="001-private-inventory" deviceset="RESISTOR" device="0204/2V" package3d_urn="urn:adsk.eagle:package:23495/1" value="4K7"/>
-<part name="C1" library="001-private-inventory" deviceset="CAPACITOR_1" device="025-024X044" package3d_urn="urn:adsk.eagle:package:23630/1" value="10nF"/>
-<part name="C2" library="001-private-inventory" deviceset="CAPACITOR_1" device="025-024X044" package3d_urn="urn:adsk.eagle:package:23630/1" value="10nF"/>
-<part name="R5" library="001-private-inventory" deviceset="RESISTOR" device="0204/2V" package3d_urn="urn:adsk.eagle:package:23495/1" value="82K"/>
+<part name="R1" library="006-rcl" library_urn="urn:adsk.eagle:library:5746079" deviceset="RESISTOR" device="0204/2V" package3d_urn="urn:adsk.eagle:package:5803065/3" value="10K"/>
+<part name="R2" library="006-rcl" library_urn="urn:adsk.eagle:library:5746079" deviceset="RESISTOR" device="0204/2V" package3d_urn="urn:adsk.eagle:package:5803065/3" value="4K7"/>
+<part name="R3" library="006-rcl" library_urn="urn:adsk.eagle:library:5746079" deviceset="RESISTOR" device="0204/2V" package3d_urn="urn:adsk.eagle:package:5803065/3" value="4K7"/>
+<part name="C1" library="006-rcl" library_urn="urn:adsk.eagle:library:5746079" deviceset="CAPACITOR_1" device="025-024X044" package3d_urn="urn:adsk.eagle:package:5815137/3" value="10nF"/>
+<part name="C2" library="006-rcl" library_urn="urn:adsk.eagle:library:5746079" deviceset="CAPACITOR_1" device="025-024X044" package3d_urn="urn:adsk.eagle:package:5815137/3" value="10nF"/>
+<part name="R5" library="006-rcl" library_urn="urn:adsk.eagle:library:5746079" deviceset="RESISTOR" device="0204/2V" package3d_urn="urn:adsk.eagle:package:5803065/3" value="82K"/>
 <part name="SUPPLY2" library="SparkFun-PowerSymbols" library_urn="urn:adsk.eagle:library:530" deviceset="5V" device=""/>
 <part name="GND1" library="SparkFun-PowerSymbols" library_urn="urn:adsk.eagle:library:530" deviceset="GND" device=""/>
 <part name="J2" library="001-private-inventory" deviceset="CONN_05" device="1X05LA" package3d_urn="urn:adsk.eagle:package:22467/2"/>
-<part name="R4" library="001-private-inventory" deviceset="RESISTOR" device="0204/2V" package3d_urn="urn:adsk.eagle:package:23495/1" value="82K"/>
+<part name="R4" library="006-rcl" library_urn="urn:adsk.eagle:library:5746079" deviceset="RESISTOR" device="0204/2V" package3d_urn="urn:adsk.eagle:package:5803065/3" value="82K"/>
 <part name="S2" library="010-inputs" library_urn="urn:adsk.eagle:library:5754152" deviceset="ENCODER_SWITCH" device="" package3d_urn="urn:adsk.eagle:package:5746065/8"/>
 </parts>
