File: type2/tht/encoder-switch-type2-tht.brd (EAGLE design)
At the start: 26 x 23.6 mm, 7 parts

Commit message: STEP files added, modified modules updated
Parts:
- C3, C4: device 001-private-inventory:C025-024X044 -> 006-rcl:C025-024X044
- R6, R7, R8: device 001-private-inventory:0204V -> 006-rcl:0204V
Changed lines of the file:
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@@
 <drawing>
 <settings>
-<setting alwaysvectorfont="no"/>
+<setting alwaysvectorfont="yes"/>
 <setting verticaltext="up"/>
 </settings>
@@
 </layers>
 <board>
+<fusionsync huburn="a.cGVyc29uYWw6dWUyYTlhNjVh" projecturn="a.cGVyc29uYWw6dWUyYTlhNjVhIzIwMTgwOTEwMTQ4MDIxNzUx" f3durn="urn:adsk.wipprod:dm.lineage:_eLT2Ce7Q7GKrSjA4S3OYA" pcbguid="997057d5-6aff-4fc7-9c01-482d86f6817f" lastpulledtime="" lastsyncedchangeguid="998c9308-7626-641b-329c-006641510251"/>
 <plain>
 <wire x1="24.765" y1="-1.905" x2="-1.27" y2="-1.905" width="0.1524" layer="20"/>
@@
 </autorouter>
 <elements>
-<element name="C3" library="001-private-inventory" package="C025-024X044" package3d_urn="urn:adsk.eagle:package:23630/1" value="100nF" x="18.288" y="17.907" rot="R180">
+<element name="C3" library="006-rcl" library_urn="urn:adsk.eagle:library:5746079" package="C025-024X044" package3d_urn="urn:adsk.eagle:package:5815137/3" value="100nF" x="18.288" y="17.907" rot="R180">
 <attribute name="NAME" x="19.304" y="20.828" size="1.27" layer="25" ratio="10" rot="R180"/>
 <attribute name="SPICEPREFIX" value="C" x="18.288" y="17.907" size="1.778" layer="27" rot="R180" display="off"/>
 </element>
-<element name="C4" library="001-private-inventory" package="C025-024X044" package3d_urn="urn:adsk.eagle:package:23630/1" value="100nF" x="10.033" y="1.905" rot="R180">
+<element name="C4" library="006-rcl" library_urn="urn:adsk.eagle:library:5746079" package="C025-024X044" package3d_urn="urn:adsk.eagle:package:5815137/3" value="100nF" x="10.033" y="1.905" rot="R180">
 <attribute name="NAME" x="11.049" y="0.381" size="1.27" layer="25" ratio="10" rot="R180"/>
 <attribute name="SPICEPREFIX" value="C" x="10.033" y="1.905" size="1.778" layer="27" rot="R180" display="off"/>
@@
 <attribute name="VALUE" x="1.397" y="8.636" size="0.6096" layer="27" font="vector" ratio="20" rot="R90"/>
 </element>
-<element name="R6" library="001-private-inventory" package="0204V" package3d_urn="urn:adsk.eagle:package:23495/1" value="10K" x="3.429" y="2.54" rot="R180">
+<element name="R6" library="006-rcl" library_urn="urn:adsk.eagle:library:5746079" package="0204V" package3d_urn="urn:adsk.eagle:package:5803065/3" value="10K" x="3.429" y="2.54" rot="R180">
 <attribute name="NAME" x="4.5466" y="1.2446" size="1.27" layer="25" ratio="10" rot="R180"/>
 <attribute name="POWER" value="0.25-0.6 W" x="3.429" y="2.54" size="1.778" layer="27" rot="R180" display="off"/>
 <attribute name="SPICEPREFIX" value="R" x="3.429" y="2.54" size="1.778" layer="27" rot="R180" display="off"/>
 </element>
-<element name="R7" library="001-private-inventory" package="0204V" package3d_urn="urn:adsk.eagle:package:23495/1" value="27K" x="21.717" y="16.637" rot="R90">
+<element name="R7" library="006-rcl" library_urn="urn:adsk.eagle:library:5746079" package="0204V" package3d_urn="urn:adsk.eagle:package:5803065/3" value="27K" x="21.717" y="16.637" rot="R90">
 <attribute name="NAME" x="22.9616" y="20.4216" size="1.27" layer="25" ratio="10" rot="R180"/>
 <attribute name="POWER" value="0.25-0.6 W" x="21.717" y="16.637" size="1.778" layer="27" rot="R90" display="off"/>
 <attribute name="SPICEPREFIX" value="R" x="21.717" y="16.637" size="1.778" layer="27" rot="R90" display="off"/>
 </element>
-<element name="R8" library="001-private-inventory" package="0204V" package3d_urn="urn:adsk.eagle:package:23495/1" value="27K" x="18.034" y="2.286" rot="R180">
+<element name="R8" library="006-rcl" library_urn="urn:adsk.eagle:library:5746079" package="0204V" package3d_urn="urn:adsk.eagle:package:5803065/3" value="27K" x="18.034" y="2.286" rot="R180">
 <attribute name="NAME" x="19.1516" y="0.8636" size="1.27" layer="25" ratio="10" rot="R180"/>
 <attribute name="POWER" value="0.25-0.6 W" x="18.034" y="2.286" size="1.778" layer="27" rot="R180" display="off"/>
@@
 </note>
 <note version="8.3" severity="warning">
+Since Version 8.3, EAGLE supports Fusion synchronisation.
+This feature will not be available in this version and saving
+the document will break the link to the Fusion PCB feature.
+</note>
+<note version="8.3" severity="warning">
