File: type2/tht/encoder-switch-type2-tht.sch (EAGLE design)
At the start: 7 parts

Commit message: STEP files added, modified modules updated
Parts:
- C3, C4: device 001-private-inventory:CAPACITOR_1025-024X044 -> 006-rcl:CAPACITOR_1025-024X044
- R6, R7, R8: device 001-private-inventory:RESISTOR0204/2V -> 006-rcl:RESISTOR0204/2V
Changed lines of the file:
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@@
 </classes>
 <parts>
-<part name="R6" library="001-private-inventory" deviceset="RESISTOR" device="0204/2V" package3d_urn="urn:adsk.eagle:package:23495/1" value="10K"/>
-<part name="R7" library="001-private-inventory" deviceset="RESISTOR" device="0204/2V" package3d_urn="urn:adsk.eagle:package:23495/1" value="27K"/>
-<part name="R8" library="001-private-inventory" deviceset="RESISTOR" device="0204/2V" package3d_urn="urn:adsk.eagle:package:23495/1" value="27K"/>
-<part name="C3" library="001-private-inventory" deviceset="CAPACITOR_1" device="025-024X044" package3d_urn="urn:adsk.eagle:package:23630/1" value="100nF"/>
-<part name="C4" library="001-private-inventory" deviceset="CAPACITOR_1" device="025-024X044" package3d_urn="urn:adsk.eagle:package:23630/1" value="100nF"/>
+<part name="R6" library="006-rcl" library_urn="urn:adsk.eagle:library:5746079" deviceset="RESISTOR" device="0204/2V" package3d_urn="urn:adsk.eagle:package:5803065/3" value="10K"/>
+<part name="R7" library="006-rcl" library_urn="urn:adsk.eagle:library:5746079" deviceset="RESISTOR" device="0204/2V" package3d_urn="urn:adsk.eagle:package:5803065/3" value="27K"/>
+<part name="R8" library="006-rcl" library_urn="urn:adsk.eagle:library:5746079" deviceset="RESISTOR" device="0204/2V" package3d_urn="urn:adsk.eagle:package:5803065/3" value="27K"/>
+<part name="C3" library="006-rcl" library_urn="urn:adsk.eagle:library:5746079" deviceset="CAPACITOR_1" device="025-024X044" package3d_urn="urn:adsk.eagle:package:5815137/3" value="100nF"/>
+<part name="C4" library="006-rcl" library_urn="urn:adsk.eagle:library:5746079" deviceset="CAPACITOR_1" device="025-024X044" package3d_urn="urn:adsk.eagle:package:5815137/3" value="100nF"/>
 <part name="SUPPLY1" library="SparkFun-PowerSymbols" library_urn="urn:adsk.eagle:library:530" deviceset="5V" device=""/>
 <part name="GND2" library="SparkFun-PowerSymbols" library_urn="urn:adsk.eagle:library:530" deviceset="GND" device=""/>
@@
 packages will not be understood (or retained) with this version.
 </note>
+<note version="8.4" severity="warning">
+Since Version 8.4, EAGLE supports properties for SPICE simulation.
+Probes in schematics and SPICE mapping objects found in parts and library devices
+will not be understood with this version. Update EAGLE to the latest version
+for full support of SPICE simulation.
+</note>
 </compatibility>
